Commit message: Init commit

File: models/iiwa_on_structure.urdf.xacro (robot description, xacro)
@@ -31,5 +31,5 @@
   <!--iiwa-->
   <xacro:iiwa7 hardware_interface="EffortJointInterface" robot_name="iiwa" parent="structure_main_link" collision_postfix="$(arg collision_postfix)">
-    <origin xyz="-0.75 0.24 1.92" rpy="3.14159 0 ${3.14159/2}"/>
+    <origin xyz="-0.75 0.24 1.92" rpy="3.14159 0 ${-3.14159/2}"/>
   </xacro:iiwa7>
 </robot>
